File: PCB-trace-tests/4-layer-microstrip-osh-v2.sch (EAGLE design)
At the start: 10 parts

Commit message: checkpoint
Parts:
- removed J10, J3, J4, J5, J6, J7, J8, J9: (no value), sma_footprint_2l:SMA-EDGE-LAUNCH4L-4020-TAPER-FIXED
- J1, J2: value (none) -> SMA-CINCH-142-0761-881; device sma_footprint_2l:SMA-EDGE-LAUNCH4L-4020-TAPER-FIXED -> yapo:SMA-CINCH-142-0761-881
Connections:
- removed net N$2: J3.CENTER, J4.CENTER
- removed net N$3 (its old number): J5.CENTER, J6.CENTER
- removed net N$4: J7.CENTER, J8.CENTER
- removed net N$5: J10.CENTER, J9.CENTER
- net GND: no longer J10.SHIELD, J3.SHIELD, J4.SHIELD, J5.SHIELD, J6.SHIELD, J7.SHIELD, J8.SHIELD, J9.SHIELD
Other:
- moved on the sheet: J1, J2
Changed lines of the file:
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@@
 <class number="0" name="default" width="0" drill="0">
 </class>
-<class number="1" name="13-5" width="0.3429" drill="0">
-</class>
-<class number="2" name="13-75" width="0.34925" drill="0">
-</class>
-<class number="3" name="14-00" width="0.3556" drill="0">
-</class>
-<class number="4" name="14-25" width="0.36195" drill="0">
-</class>
-<class number="5" name="14-50" width="0.3683" drill="0">
+<class number="1" name="12.5-6-cpwg" width="0.3175" drill="0">
+<clearance class="1" value="0.1524"/>
 </class>
 </classes>
 <parts>
-<part name="J1" library="sma_footprint_2l" deviceset="SMA-EDGE-LAUNCH" device="4L-4020-TAPER-FIXED"/>
-<part name="J2" library="sma_footprint_2l" deviceset="SMA-EDGE-LAUNCH" device="4L-4020-TAPER-FIXED"/>
-<part name="U$1" library="yapo" deviceset="GND" device=""/>
-<part name="U$2" library="yapo" deviceset="GND" device=""/>
-<part name="J3" library="sma_footprint_2l" deviceset="SMA-EDGE-LAUNCH" device="4L-4020-TAPER-FIXED"/>
-<part name="J4" library="sma_footprint_2l" deviceset="SMA-EDGE-LAUNCH" device="4L-4020-TAPER-FIXED"/>
-<part name="U$3" library="yapo" deviceset="GND" device=""/>
-<part name="U$4" library="yapo" deviceset="GND" device=""/>
-<part name="J5" library="sma_footprint_2l" deviceset="SMA-EDGE-LAUNCH" device="4L-4020-TAPER-FIXED"/>
-<part name="J6" library="sma_footprint_2l" deviceset="SMA-EDGE-LAUNCH" device="4L-4020-TAPER-FIXED"/>
 <part name="U$5" library="yapo" deviceset="GND" device=""/>
 <part name="U$6" library="yapo" deviceset="GND" device=""/>
-<part name="J7" library="sma_footprint_2l" deviceset="SMA-EDGE-LAUNCH" device="4L-4020-TAPER-FIXED"/>
-<part name="J8" library="sma_footprint_2l" deviceset="SMA-EDGE-LAUNCH" device="4L-4020-TAPER-FIXED"/>
-<part name="U$7" library="yapo" deviceset="GND" device=""/>
-<part name="U$8" library="yapo" deviceset="GND" device=""/>
-<part name="J9" library="sma_footprint_2l" deviceset="SMA-EDGE-LAUNCH" device="4L-4020-TAPER-FIXED"/>
-<part name="J10" library="sma_footprint_2l" deviceset="SMA-EDGE-LAUNCH" device="4L-4020-TAPER-FIXED"/>
-<part name="U$9" library="yapo" deviceset="GND" device=""/>
-<part name="U$10" library="yapo" deviceset="GND" device=""/>
+<part name="J1" library="yapo" deviceset="SMA-CINCH-142-0761-881" device=""/>
+<part name="J2" library="yapo" deviceset="SMA-CINCH-142-0761-881" device=""/>
 </parts>
 <sheets>
@@
 </plain>
 <instances>
-<instance part="J1" gate="G$1" x="144.78" y="53.34" smashed="yes">
-<attribute name="NAME" x="149.86" y="58.42" size="1.27" layer="95"/>
-<attribute name="VALUE" x="149.86" y="55.88" size="1.27" layer="96"/>
-</instance>
-<instance part="J2" gate="G$1" x="96.52" y="53.34" smashed="yes" rot="MR0">
-<attribute name="NAME" x="91.44" y="58.42" size="1.27" layer="95" rot="MR0"/>
-<attribute name="VALUE" x="91.44" y="55.88" size="1.27" layer="96" rot="MR0"/>
-</instance>
-<instance part="U$1" gate="G$1" x="96.52" y="43.18" smashed="yes"/>
-<instance part="U$2" gate="G$1" x="144.78" y="43.18" smashed="yes"/>
-<instance part="J3" gate="G$1" x="144.78" y="27.94" smashed="yes">
-<attribute name="NAME" x="149.86" y="33.02" size="1.27" layer="95"/>
-<attribute name="VALUE" x="149.86" y="30.48" size="1.27" layer="96"/>
-</instance>
-<instance part="J4" gate="G$1" x="96.52" y="27.94" smashed="yes" rot="MR0">
-<attribute name="NAME" x="91.44" y="33.02" size="1.27" layer="95" rot="MR0"/>
-<attribute name="VALUE" x="91.44" y="30.48" size="1.27" layer="96" rot="MR0"/>
-</instance>
-<instance part="U$3" gate="G$1" x="96.52" y="17.78" smashed="yes"/>
-<instance part="U$4" gate="G$1" x="144.78" y="17.78" smashed="yes"/>
-<instance part="J5" gate="G$1" x="144.78" y="2.54" smashed="yes">
+<instance part="U$5" gate="G$1" x="96.52" y="-7.62" smashed="yes"/>
+<instance part="U$6" gate="G$1" x="144.78" y="-7.62" smashed="yes"/>
+<instance part="J1" gate="G$1" x="144.78" y="2.54" smashed="yes">
 <attribute name="NAME" x="149.86" y="7.62" size="1.27" layer="95"/>
 <attribute name="VALUE" x="149.86" y="5.08" size="1.27" layer="96"/>
 </instance>
-<instance part="J6" gate="G$1" x="96.52" y="2.54" smashed="yes" rot="MR0">
+<instance part="J2" gate="G$1" x="96.52" y="2.54" smashed="yes" rot="MR0">
 <attribute name="NAME" x="91.44" y="7.62" size="1.27" layer="95" rot="MR0"/>
 <attribute name="VALUE" x="91.44" y="5.08" size="1.27" layer="96" rot="MR0"/>
 </instance>
-<instance part="U$5" gate="G$1" x="96.52" y="-7.62" smashed="yes"/>
-<instance part="U$6" gate="G$1" x="144.78" y="-7.62" smashed="yes"/>
-<instance part="J7" gate="G$1" x="144.78" y="78.74" smashed="yes">
-<attribute name="NAME" x="149.86" y="83.82" size="1.27" layer="95"/>
-<attribute name="VALUE" x="149.86" y="81.28" size="1.27" layer="96"/>
-</instance>
-<instance part="J8" gate="G$1" x="96.52" y="78.74" smashed="yes" rot="MR0">
-<attribute name="NAME" x="91.44" y="83.82" size="1.27" layer="95" rot="MR0"/>
-<attribute name="VALUE" x="91.44" y="81.28" size="1.27" layer="96" rot="MR0"/>
-</instance>
-<instance part="U$7" gate="G$1" x="96.52" y="68.58" smashed="yes"/>
-<instance part="U$8" gate="G$1" x="144.78" y="68.58" smashed="yes"/>
-<instance part="J9" gate="G$1" x="144.78" y="101.6" smashed="yes">
-<attribute name="NAME" x="149.86" y="106.68" size="1.27" layer="95"/>
-<attribute name="VALUE" x="149.86" y="104.14" size="1.27" layer="96"/>
-</instance>
-<instance part="J10" gate="G$1" x="96.52" y="101.6" smashed="yes" rot="MR0">
-<attribute name="NAME" x="91.44" y="106.68" size="1.27" layer="95" rot="MR0"/>
-<attribute name="VALUE" x="91.44" y="104.14" size="1.27" layer="96" rot="MR0"/>
-</instance>
-<instance part="U$9" gate="G$1" x="96.52" y="91.44" smashed="yes"/>
-<instance part="U$10" gate="G$1" x="144.78" y="91.44" smashed="yes"/>
 </instances>
 <busses>
 </busses>
 <nets>
+<net name="N$3" class="1">
+<segment>
+<wire x1="104.14" y1="2.54" x2="137.16" y2="2.54" width="0.1524" layer="91"/>
+<pinref part="J1" gate="G$1" pin="CENTER"/>
+<pinref part="J2" gate="G$1" pin="CENTER"/>
+</segment>
+</net>
 <net name="GND" class="0">
 <segment>
-<pinref part="J2" gate="G$1" pin="SHIELD"/>
-<pinref part="U$1" gate="G$1" pin="GND"/>
+<pinref part="U$6" gate="G$1" pin="GND"/>
+<pinref part="J1" gate="G$1" pin="SHIELD"/>
 </segment>
 <segment>
-<pinref part="J1" gate="G$1" pin="SHIELD"/>
-<pinref part="U$2" gate="G$1" pin="GND"/>
-</segment>
-<segment>
-<pinref part="J4" gate="G$1" pin="SHIELD"/>
-<pinref part="U$3" gate="G$1" pin="GND"/>
-</segment>
-<segment>
-<pinref part="J3" gate="G$1" pin="SHIELD"/>
-<pinref part="U$4" gate="G$1" pin="GND"/>
-</segment>
-<segment>
-<pinref part="J6" gate="G$1" pin="SHIELD"/>
 <pinref part="U$5" gate="G$1" pin="GND"/>
-</segment>
-<segment>
-<pinref part="J5" gate="G$1" pin="SHIELD"/>
-<pinref part="U$6" gate="G$1" pin="GND"/>
-</segment>
-<segment>
-<pinref part="J8" gate="G$1" pin="SHIELD"/>
-<pinref part="U$7" gate="G$1" pin="GND"/>
-</segment>
-<segment>
-<pinref part="J7" gate="G$1" pin="SHIELD"/>
-<pinref part="U$8" gate="G$1" pin="GND"/>
-</segment>
-<segment>
-<pinref part="J10" gate="G$1" pin="SHIELD"/>
-<pinref part="U$9" gate="G$1" pin="GND"/>
-</segment>
-<segment>
-<pinref part="J9" gate="G$1" pin="SHIELD"/>
-<pinref part="U$10" gate="G$1" pin="GND"/>
+<pinref part="J2" gate="G$1" pin="SHIELD"/>
 </segment>
 </net>
-<net name="N$1" class="1">
-<segment>
-<pinref part="J2" gate="G$1" pin="CENTER"/>
-<pinref part="J1" gate="G$1" pin="CENTER"/>
-<wire x1="104.14" y1="53.34" x2="137.16" y2="53.34" width="0.1524" layer="91"/>
-</segment>
-</net>
-<net name="N$2" class="2">
-<segment>
-<pinref part="J4" gate="G$1" pin="CENTER"/>
-<pinref part="J3" gate="G$1" pin="CENTER"/>
-<wire x1="104.14" y1="27.94" x2="137.16" y2="27.94" width="0.1524" layer="91"/>
-</segment>
-</net>
-<net name="N$3" class="3">
-<segment>
-<pinref part="J6" gate="G$1" pin="CENTER"/>
-<pinref part="J5" gate="G$1" pin="CENTER"/>
-<wire x1="104.14" y1="2.54" x2="137.16" y2="2.54" width="0.1524" layer="91"/>
-</segment>
-</net>
-<net name="N$4" class="4">
-<segment>
-<pinref part="J8" gate="G$1" pin="CENTER"/>
-<pinref part="J7" gate="G$1" pin="CENTER"/>
-<wire x1="104.14" y1="78.74" x2="137.16" y2="78.74" width="0.1524" layer="91"/>
-</segment>
-</net>
-<net name="N$5" class="5">
-<segment>
-<pinref part="J10" gate="G$1" pin="CENTER"/>
-<pinref part="J9" gate="G$1" pin="CENTER"/>
-<wire x1="104.14" y1="101.6" x2="137.16" y2="101.6" width="0.1524" layer="91"/>
-</segment>
-</net>
