File: ADCMP582-sampler/adcmp582-sampler.sch (EAGLE design)
At the start: 68 parts, among them IC12 MC79M05, IC13 MC78M05, IC2 MC100EPT21, IC3 SY89296U, IC6 AD711

Commit message: checkpoint
Connections:
- removed net ACQUIRED: IC14.!Q!
- removed net N$39: IC14.R, IC15.!Q!
- removed net TRIG-EN: IC14.CP
- net +3.3V: now also IC14.R; no longer IC14.D
- net N$40: now also IC14.CP
Changed lines of the file:
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@@
 <?xml version="1.0" encoding="utf-8"?>
 <!DOCTYPE eagle SYSTEM "eagle.dtd">
-<eagle version="9.4.1">
+<eagle version="9.4.2">
 <drawing>
 <settings>
@@
 <pinref part="U$89" gate="G$1" pin="+3.3V"/>
 <wire x1="30.48" y1="111.76" x2="30.48" y2="109.22" width="0.1524" layer="91"/>
-<pinref part="IC14" gate="G$1" pin="D"/>
-<wire x1="17.78" y1="93.98" x2="12.7" y2="93.98" width="0.1524" layer="91"/>
-<wire x1="12.7" y1="93.98" x2="12.7" y2="101.6" width="0.1524" layer="91"/>
 <wire x1="12.7" y1="101.6" x2="12.7" y2="109.22" width="0.1524" layer="91"/>
 <wire x1="12.7" y1="109.22" x2="30.48" y2="109.22" width="0.1524" layer="91"/>
@@
 <pinref part="IC14" gate="G$1" pin="S"/>
 <wire x1="17.78" y1="101.6" x2="12.7" y2="101.6" width="0.1524" layer="91"/>
+<pinref part="IC14" gate="G$1" pin="R"/>
+<wire x1="17.78" y1="81.28" x2="12.7" y2="81.28" width="0.1524" layer="91"/>
+<wire x1="12.7" y1="81.28" x2="12.7" y2="101.6" width="0.1524" layer="91"/>
 <junction x="12.7" y="101.6"/>
 </segment>
@@
 </segment>
 </net>
-<net name="N$39" class="0">
-<segment>
-<pinref part="IC15" gate="G$1" pin="!Q!"/>
-<wire x1="106.68" y1="86.36" x2="111.76" y2="86.36" width="0.1524" layer="91"/>
-<wire x1="111.76" y1="86.36" x2="111.76" y2="66.04" width="0.1524" layer="91"/>
-<wire x1="111.76" y1="66.04" x2="12.7" y2="66.04" width="0.1524" layer="91"/>
-<wire x1="12.7" y1="66.04" x2="12.7" y2="81.28" width="0.1524" layer="91"/>
-<pinref part="IC14" gate="G$1" pin="R"/>
-<wire x1="12.7" y1="81.28" x2="17.78" y2="81.28" width="0.1524" layer="91"/>
-</segment>
-</net>
 <net name="N$40" class="0">
 <segment>
@@
 <wire x1="81.28" y1="88.9" x2="68.58" y2="88.9" width="0.1524" layer="91"/>
 <wire x1="68.58" y1="88.9" x2="68.58" y2="60.96" width="0.1524" layer="91"/>
-<wire x1="68.58" y1="60.96" x2="-2.54" y2="60.96" width="0.1524" layer="91"/>
-</segment>
-</net>
-<net name="TRIG-EN" class="0">
-<segment>
+<wire x1="68.58" y1="60.96" x2="2.54" y2="60.96" width="0.1524" layer="91"/>
+<wire x1="2.54" y1="60.96" x2="2.54" y2="88.9" width="0.1524" layer="91"/>
+<junction x="2.54" y="60.96"/>
 <pinref part="IC14" gate="G$1" pin="CP"/>
-<wire x1="17.78" y1="88.9" x2="-2.54" y2="88.9" width="0.1524" layer="91"/>
-<label x="-2.54" y="88.9" size="1.778" layer="95" rot="R180" xref="yes"/>
+<wire x1="2.54" y1="88.9" x2="17.78" y2="88.9" width="0.1524" layer="91"/>
+<wire x1="2.54" y1="60.96" x2="-30.48" y2="60.96" width="0.1524" layer="91"/>
 </segment>
 </net>
@@
 </segment>
 </net>
-<net name="ACQUIRED" class="0">
-<segment>
-<pinref part="IC14" gate="G$1" pin="!Q!"/>
-<wire x1="43.18" y1="86.36" x2="48.26" y2="86.36" width="0.1524" layer="91"/>
-<label x="48.26" y="86.36" size="1.778" layer="95" xref="yes"/>
-</segment>
-</net>

Commit message: checkpoint
Parts:
- removed IC14, IC15: (no value), yapo:74LVC2G74
- removed U$34: 74LVC1G04, yapo:74LVC1G04
- removed U$46, U$47, U$48: PAD50MIL, yapo:PAD50MIL
- added C21, C22, C23, C24, C25, C26, C27, C28, C30, C31, C32, C33, C34, C35, C36, C37, C38: (no value), yapo:C0603
- added C29: (no value), yapo:C1206
- added J2: ICSP_HEADER, yapo:ICSP_HEADER
- added J3, J4: (no value), sma_footprint_2l:SMA-EDGE-LAUNCH4L-4020-TAPER-FIXED
- added J5, J6, J7: (no value), yapo:HEADER_2PINSCREW-TERM
- added P1, P2, P3, P4, P5, P6, P7: ICSP_PAD, yapo:ICSP_PAD
- added R17, R18, R29, R30, R31, R32, R33: (no value), yapo:R0603
- added R19, R20, R25, R27, R28: (no value), yapo:R0402
- added U$140: 74LVC1G04, yapo:74LVC1G04
- added U$36: (no value), yapo:74LVC1G17
- added U$54: HEADER_3PIN, yapo:HEADER_3PIN
- added U$57, U$86, U$87, U$91, U$92, U$93, U$94, U$95, U$96, U$98: NO_CONNECT, yapo:NO_CONNECT
- added U$88: LED_0603, yapo:LED_0603
- added X1: (no value), yapo:XTAL_OSC
- C10, C11, C12, C13, C6, C7, C8, C9: device yapo:C0603 -> yapo:C1206
- IC4: device yapo:MC100LVELT20 -> yapo:PIC16F15376
- IC5: device yapo:MCP48X1 -> yapo:ADA4000
- IC6: value AD711 -> (none); device yapo:AD711 -> yapo:MC100LVELT20
- IC8: device yapo:74XX595 -> yapo:SI53360TSSOP16
- IC9: device yapo:74XX595 -> yapo:74LVC1G79
- J1: device yapo:SMA_END_LAUNCH4L -> sma_footprint_2l:SMA-EDGE-LAUNCH4L-4020-TAPER-FIXED
- U$90: value 74LVC1G04 -> NO_CONNECT; device yapo:74LVC1G04 -> yapo:NO_CONNECT
Connections:
- net LE_P renamed LE_P1
- net N$1 renamed INPUT
- removed net N$28: C9.P$2, IC11.IN
- removed net N$29: C6.P$2, IC10.OUT
- removed net N$30: C8.P$2, IC11.OUT
- removed net N$31: C11.P$2, IC12.IN
- removed net N$32: C10.P$2, IC12.OUT
- removed net N$33: C13.P$2, IC13.IN
- removed net N$34: C12.P$2, IC13.OUT
- removed net N$40: IC14.CP, IC15.CP
- removed net RCLK: IC8.RCLK, IC9.RCLK
- removed net SER: IC8.SER
- removed net SRCLK: IC8.SRCLK, IC9.SRCLK
- removed net TUNE-!CS!: IC5.!CS!
- removed net TUNE-SCK: IC5.SCK
- removed net TUNE-SDI: IC5.SDI
- new net !LDAC!: IC1.!LDAC!, IC4.RC5
- new net !MCLR!: IC4.VPP/!MCLR!/RE3, J2.!MCLR!/VPP, R17.P$4
- new net CLK-SEL: IC4.RE2, IC8.CLK_SEL
- new net CLOCK-OUT: J4.CENTER, R19.P$4, R20.P$4, R25.P$4, R27.P$4, R28.P$4
- new net COMP-CLK: IC4.RB4, IC8.Q5
- new net COMP-OUT: IC4.RB3, IC9.Q
- new net COMP-REG-CLK: IC8.Q3, U$140.IN
- new net ICSPCLK: IC4.ICSPCLK/RB6, J2.ICSPCLK
- new net ICSPDAT: IC4.ICSPDAT/RB7, J2.ICSPDAT
- new net N$1: R31.P$3, U$36.OUT
- new net N$26: R33.P$4, U$88.A
- new net N$39: IC8.Q6, R27.P$3
- new net N$41: IC8.Q2, R25.P$3
- new net N$43: IC8.Q0, R19.P$3
- new net N$44: IC4.RC6, R29.P$3
- new net N$45: IC4.RC7, R30.P$3
- new net N$47: IC4.RC1, U$57.P$1
- new net N$48: IC4.RC2, U$86.P$1
- new net N$49: IC4.RC3, U$87.P$1
- new net N$52: IC3.FTUNE, U$90.P$1
- new net N$53: IC4.RA0, U$91.P$1
- new net N$54: IC4.RA1, U$92.P$1
- new net N$55: IC4.RA2, U$93.P$1
- new net N$56: IC4.RA3, U$94.P$1
- new net N$57: IC4.RA4, U$95.P$1
- new net N$58: IC4.RA5, U$96.P$1
- new net N$60: IC4.RA6, U$98.P$1
- new net RX: R30.P$4, U$54.3
- new net SAMPLE-CLOCK: IC4.RC0, IC8.CLK1
- new net TRIGGER: J3.CENTER, U$36.IN
- new net TX: R29.P$4, U$54.1
- new net VCC2: C22.P$2, C23.P$2, C24.P$2, C36.P$2, C37.P$2, C38.P$2, C8.P$2, IC11.OUT, IC4.VDD@1, IC4.VDD@2, IC9.VCC, J2.VDD, P6.P$1, R17.P$3, U$140.VCC, U$36.VCC, X1.VCC
- new net VDAC: C5.P$2, IC1.VOUT, IC5G$1.-, P2.P$1
- new net VIN+5: C13.P$2, IC13.IN, J6.1
- new net VIN-5: C11.P$2, IC12.IN, J5.1
- new net VIN3.3: C7.P$2, C9.P$2, IC10.IN, IC11.IN, J7.1
- net +3.3V: now also C19.P$2, C21.P$2, C27.P$2, C28.P$2, C3.P$2, C30.P$2, C31.P$2, C32.P$2, C33.P$2, C6.P$2, IC10.OUT, IC6.VCC, IC8.OE, IC8.VDD, P5.P$1; no longer IC14.R, IC14.S, IC14.VCC, IC15.R, IC15.S, IC15.VCC, IC4.VCC, IC5.!SHDN!, IC5.VDD, IC8.!SRCLR!, IC8.VCC, IC9.!SRCLR!, IC9.VCC, U$34.VCC, U$90.VCC
- net +5V: now also C12.P$2, C25.P$2, C29.P$2, C34.P$2, IC13.OUT, IC5G$2.V+, P4.P$1; no longer IC6.+V
- net -5V: now also C10.P$2, C26.P$2, C35.P$2, IC12.OUT, IC5G$2.GND, P3.P$1; no longer C19.P$2, IC6.-V, U$48.P$1
- net D0: now also IC4.RD0; no longer IC8.QH
- net D1: now also IC4.RD1; no longer IC8.QG
- net D2: now also IC4.RD2; no longer IC8.QF
- net D3: now also IC4.RD3; no longer IC8.QE
- net D4: now also IC4.RD4; no longer IC8.QD
- net D5: now also IC4.RD5; no longer IC8.QC
- net D6: now also IC4.RD6; no longer IC8.QB
- net D7: now also IC4.RD7; no longer IC8.QA
- net D8: now also IC4.RE0; no longer IC9.QC
- net D9: now also IC4.RE1; no longer IC9.QB
- net GND: now also C21.P$1, C22.P$1, C23.P$1, C24.P$1, C25.P$1, C26.P$1, C27.P$1, C28.P$1, C29.P$1, C30.P$1, C31.P$1, C32.P$1, C33.P$1, C34.P$1, C35.P$1, C36.P$1, C37.P$1, C38.P$1, IC4.VSS@1, IC4.VSS@2, IC6.GND, J2.VSS, J3.SHIELD, J4.SHIELD, J5.2, J6.2, J7.2, U$140.GND, U$36.GND, U$54.2, U$88.C, X1.GND; no longer IC1.!LDAC!, IC14.GND, IC15.GND, IC4.GND, IC5.!LDAC!, IC5.VSS, IC8.!OE!, IC9.!OE!, U$34.GND, U$90.GND
- net N$16: now also IC3.IN, IC6.Q; no longer IC3./IN, IC4.Q
- net N$17: now also IC2.Q, R32.P$3; no longer IC3.IN, IC4.!Q!, R22.P$4, R24.P$3
- net N$18: now also IC8.Q4, R18.P$3; no longer C3.P$2, IC3.FTUNE, IC5.VOUT
- net N$19: now also IC9.CLK, U$140.OUT; no longer IC2.Q, U$34.IN
- net N$20: now also IC5G$1.+; no longer IC6.IN-
- net N$21: now also IC5G$1.OUT; no longer IC6.OUT
- net N$22: now also IC3./IN, IC6.!Q!, R22.P$4, R24.P$3; no longer C5.P$2, IC1.VOUT, IC6.IN+
- net N$23: now also IC8.CLK0, R31.P$4; no longer IC6.NULL_A, U$47.P$1
- net N$24: now also IC4.RA7, X1.OUT; no longer IC6.NULL_B, U$46.P$1
- net N$25: now also IC4.RC4, R33.P$3; no longer IC8.SER_OUT, IC9.SER
- net N$27: now also IC9.D, R32.P$4; no longer C7.P$2, IC10.IN
- net N$36: now also IC6.D, R18.P$4; no longer IC4.D, U$90.OUT
- net N$38: now also IC8.Q7, R28.P$3; no longer IC14.Q, IC15.D
- net N$42: now also IC8.Q1, R20.P$3; no longer IC15.Q, U$90.IN
- net V2.048: now also P7.P$1
- net VREF: now also P1.P$1
- net VREF-!CS!: now also IC4.RB0
- net VREF-SCK: now also IC4.RB1
- net VREF-SDI: now also IC4.RB2
Other:
- moved on the sheet: C10, C11, C12, C13, C19, C3, C6, C7, C8, C9, IC10, IC11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

Commit message: checkpoint
Parts:
- R12: value (none) -> 20k
- R13, R14: value (none) -> 10k
Changed lines of the file:
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@@
 <grid distance="0.1" unitdist="inch" unit="inch" style="lines" multiple="1" display="no" altdistance="0.01" altunitdist="inch" altunit="inch"/>
 <layers>
-<layer number="1" name="Top" color="4" fill="1" visible="yes" active="no"/>
-<layer number="2" name="Route2" color="16" fill="1" visible="yes" active="no"/>
-<layer number="15" name="Route15" color="23" fill="1" visible="yes" active="no"/>
-<layer number="16" name="Bottom" color="1" fill="1" visible="yes" active="no"/>
-<layer number="17" name="Pads" color="2" fill="1" visible="yes" active="no"/>
-<layer number="18" name="Vias" color="2" fill="1" visible="yes" active="no"/>
-<layer number="19" name="Unrouted" color="6" fill="1" visible="yes" active="no"/>
-<layer number="20" name="Dimension" color="24" fill="1" visible="yes" active="no"/>
-<layer number="21" name="tPlace" color="7" fill="1" visible="yes" active="no"/>
-<layer number="22" name="bPlace" color="7" fill="1" visible="yes" active="no"/>
-<layer number="23" name="tOrigins" color="15" fill="1" visible="yes" active="no"/>
-<layer number="24" name="bOrigins" color="15" fill="1" visible="yes" active="no"/>
-<layer number="25" name="tNames" color="7" fill="1" visible="yes" active="no"/>
-<layer number="26" name="bNames" color="7" fill="1" visible="yes" active="no"/>
-<layer number="27" name="tValues" color="7" fill="1" visible="yes" active="no"/>
-<layer number="28" name="bValues" color="7" fill="1" visible="yes" active="no"/>
+<layer number="1" name="Top" color="4" fill="1" visible="no" active="no"/>
+<layer number="2" name="Route2" color="16" fill="1" visible="no" active="no"/>
+<layer number="15" name="Route15" color="23" fill="1" visible="no" active="no"/>
+<layer number="16" name="Bottom" color="1" fill="1" visible="no" active="no"/>
+<layer number="17" name="Pads" color="2" fill="1" visible="no" active="no"/>
+<layer number="18" name="Vias" color="2" fill="1" visible="no" active="no"/>
+<layer number="19" name="Unrouted" color="6" fill="1" visible="no" active="no"/>
+<layer number="20" name="Dimension" color="24" fill="1" visible="no" active="no"/>
+<layer number="21" name="tPlace" color="7" fill="1" visible="no" active="no"/>
+<layer number="22" name="bPlace" color="7" fill="1" visible="no" active="no"/>
+<layer number="23" name="tOrigins" color="15" fill="1" visible="no" active="no"/>
+<layer number="24" name="bOrigins" color="15" fill="1" visible="no" active="no"/>
+<layer number="25" name="tNames" color="7" fill="1" visible="no" active="no"/>
+<layer number="26" name="bNames" color="7" fill="1" visible="no" active="no"/>
+<layer number="27" name="tValues" color="7" fill="1" visible="no" active="no"/>
+<layer number="28" name="bValues" color="7" fill="1" visible="no" active="no"/>
 <layer number="29" name="tStop" color="7" fill="3" visible="no" active="no"/>
 <layer number="30" name="bStop" color="7" fill="6" visible="no" active="no"/>
@@
 <layer number="35" name="tGlue" color="7" fill="4" visible="no" active="no"/>
 <layer number="36" name="bGlue" color="7" fill="5" visible="no" active="no"/>
-<layer number="37" name="tTest" color="7" fill="1" visible="yes" active="no"/>
-<layer number="38" name="bTest" color="7" fill="1" visible="yes" active="no"/>
+<layer number="37" name="tTest" color="7" fill="1" visible="no" active="no"/>
+<layer number="38" name="bTest" color="7" fill="1" visible="no" active="no"/>
 <layer number="39" name="tKeepout" color="4" fill="11" visible="no" active="no"/>
 <layer number="40" name="bKeepout" color="1" fill="11" visible="no" active="no"/>
@@
 <layer number="44" name="Drills" color="7" fill="1" visible="no" active="no"/>
 <layer number="45" name="Holes" color="7" fill="1" visible="no" active="no"/>
-<layer number="46" name="Milling" color="3" fill="1" visible="yes" active="no"/>
-<layer number="47" name="Measures" color="7" fill="1" visible="yes" active="no"/>
-<layer number="48" name="Document" color="7" fill="1" visible="yes" active="no"/>
-<layer number="49" name="Reference" color="7" fill="1" visible="yes" active="no"/>
-<layer number="51" name="tDocu" color="7" fill="1" visible="yes" active="no"/>
-<layer number="52" name="bDocu" color="7" fill="1" visible="yes" active="no"/>
+<layer number="46" name="Milling" color="3" fill="1" visible="no" active="no"/>
+<layer number="47" name="Measures" color="7" fill="1" visible="no" active="no"/>
+<layer number="48" name="Document" color="7" fill="1" visible="no" active="no"/>
+<layer number="49" name="Reference" color="7" fill="1" visible="no" active="no"/>
+<layer number="51" name="tDocu" color="7" fill="1" visible="no" active="no"/>
+<layer number="52" name="bDocu" color="7" fill="1" visible="no" active="no"/>
 <layer number="88" name="SimResults" color="9" fill="1" visible="yes" active="yes"/>
 <layer number="89" name="SimProbes" color="9" fill="1" visible="yes" active="yes"/>
@@
 <part name="U$28" library="yapo" deviceset="NO_CONNECT" device=""/>
 <part name="U$29" library="yapo" deviceset="NO_CONNECT" device=""/>
-<part name="R12" library="yapo" deviceset="R" device="0603"/>
-<part name="R13" library="yapo" deviceset="R" device="0603"/>
-<part name="R14" library="yapo" deviceset="R" device="0603"/>
+<part name="R12" library="yapo" deviceset="R" device="0603" value="20k"/>
+<part name="R13" library="yapo" deviceset="R" device="0603" value="10k"/>
+<part name="R14" library="yapo" deviceset="R" device="0603" value="10k"/>
 <part name="IC7" library="yapo" deviceset="MCP1501" device="SOIC8"/>
 <part name="U$37" library="yapo" deviceset="GND" device=""/>
