File: lvc-strobe-generator/lvc-strobe-generator.brd (EAGLE design)
At the start: 32.4 x 22.5 mm, 17 parts

Commit message: checkpoint
Parts:
- added C7: (no value), yapo:C0603
- J1, J2, J3: device sma_footprint_2l:SMA_EDGE_LAUNCH_2L_4020_TAPER -> sma_footprint_2l:SMA_EDGE_LAUNCH_4L_4020_TAPER_FIXED
- R3: device yapo:R0603 -> yapo:0402
- moved R2 2.96 mm to (22.9, 20.7), turned to 0 degrees
- moved R1 2.84 mm to (20.1, 20.7), turned to 0 degrees
- moved C1 0.64 mm to (20.4, 19.4)
- moved C6 0.64 mm to (22.5, 19.4)
- turned C3 to 0 degrees
- turned J4 to 180 degrees
Connections:
- net +5V: now also C7.P$2
- net GND: now also C7.P$1
- net N$1: now also R3.1; no longer R3.P$1
- net N$4: now also R3.2; no longer R3.P$2
- net N$7: now also J1.P$3
- net N$8: now also J3.P$3
- net N$9: now also J2.P$3
Routing:
- net +5V: track 17.6 -> 55.1 mm
- net N$2: track 45.6 -> 58.1 mm
- added copper zone on layer 1, net +5V
- added copper zone on layer 1, net N$7
Other:
- board text added: "74LVC Strobe Gen"
- board text added: "Yapo 2019"
- board text removed: "500 ps delay?"
- board text removed: "500ps = 1488 mils"
- board text removed: "build 2-layer test pcb"
- board text removed: "clock in, differential pulse out"
- board text removed: "sma input, unterminated"
- board text removed: "sma outputs with 453 resistors"
