File: lvc-strobe-generator/lvc-strobe-generator.sch (EAGLE design)
At the start: 17 parts

Commit message: checkpoint
Parts:
- added C7: (no value), yapo:C0603
- J1, J2, J3: device sma_footprint_2l:SMA-EDGE-LAUNCH4020_TAPER -> sma_footprint_2l:SMA-EDGE-LAUNCH4L-4020-TAPER-FIXED
- R3: device yapo:R0603 -> yapo:R0402
Connections:
- net +5V: now also C7.P$2
- net GND: now also C7.P$1
Changed lines of the file:
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@@
 <?xml version="1.0" encoding="utf-8"?>
 <!DOCTYPE eagle SYSTEM "eagle.dtd">
-<eagle version="9.4.2">
+<eagle version="9.4.1">
 <drawing>
 <settings>
@@
 <part name="U$8" library="yapo" deviceset="GND" device=""/>
 <part name="U$9" library="yapo" deviceset="GND" device=""/>
-<part name="R3" library="yapo" deviceset="R" device="0603"/>
+<part name="R3" library="yapo" deviceset="R" device="0402"/>
 <part name="C2" library="yapo" deviceset="C" device=""/>
-<part name="J1" library="sma_footprint_2l" deviceset="SMA-EDGE-LAUNCH" device="4020_TAPER"/>
-<part name="J2" library="sma_footprint_2l" deviceset="SMA-EDGE-LAUNCH" device="4020_TAPER"/>
-<part name="J3" library="sma_footprint_2l" deviceset="SMA-EDGE-LAUNCH" device="4020_TAPER"/>
+<part name="J1" library="sma_footprint_2l" deviceset="SMA-EDGE-LAUNCH" device="4L-4020-TAPER-FIXED"/>
+<part name="J2" library="sma_footprint_2l" deviceset="SMA-EDGE-LAUNCH" device="4L-4020-TAPER-FIXED"/>
+<part name="J3" library="sma_footprint_2l" deviceset="SMA-EDGE-LAUNCH" device="4L-4020-TAPER-FIXED"/>
 <part name="R4" library="yapo" deviceset="R" device="0603"/>
 <part name="R5" library="yapo" deviceset="R" device="0603"/>
@@
 <part name="C6" library="yapo" deviceset="C" device=""/>
 <part name="U$21" library="yapo" deviceset="GND" device=""/>
+<part name="C7" library="yapo" deviceset="C" device="0603"/>
+<part name="U$22" library="yapo" deviceset="GND" device=""/>
+<part name="U$23" library="yapo" deviceset="+5V" device=""/>
 </parts>
 <sheets>
@@
 </instance>
 <instance part="U$21" gate="G$1" x="114.3" y="71.12" smashed="yes"/>
+<instance part="C7" gate="G$1" x="198.12" y="93.98" smashed="yes">
+<attribute name="NAME" x="200.66" y="99.06" size="1.778" layer="95" font="vector"/>
+<attribute name="VALUE" x="200.66" y="96.52" size="1.778" layer="96" font="vector"/>
+</instance>
+<instance part="U$22" gate="G$1" x="198.12" y="86.36" smashed="yes"/>
+<instance part="U$23" gate="G$1" x="198.12" y="104.14" smashed="yes">
+<attribute name="VALUE" x="199.39" y="104.14" size="1.27" layer="96"/>
+</instance>
 </instances>
 <busses>
@@
 <wire x1="187.96" y1="99.06" x2="187.96" y2="101.6" width="0.1524" layer="91"/>
 </segment>
+<segment>
+<pinref part="C7" gate="G$1" pin="P$2"/>
+<pinref part="U$23" gate="G$1" pin="+5V"/>
+<wire x1="198.12" y1="99.06" x2="198.12" y2="101.6" width="0.1524" layer="91"/>
+</segment>
 </net>
 <net name="GND" class="0">
@@
 <pinref part="C6" gate="G$1" pin="P$1"/>
 <pinref part="U$21" gate="G$1" pin="GND"/>
+</segment>
+<segment>
+<pinref part="U$22" gate="G$1" pin="GND"/>
+<pinref part="C7" gate="G$1" pin="P$1"/>
+<wire x1="198.12" y1="86.36" x2="198.12" y2="88.9" width="0.1524" layer="91"/>
 </segment>
 </net>
@@
 </segment>
 </net>
-<net name="N$7" class="2">
+<net name="N$7" class="0">
 <segment>
 <pinref part="J1" gate="G$1" pin="CENTER"/>
